File: hardware/KiCad/elephant/power.kicad_sch (KiCad schematic)
At the start: 28 parts, among them U3 LT8640, U5 74AUP1G74, U6 LM66100DCK, U7 LM66100DCK

Commit message: Tilt switch tests completed; tilt switch circuit verified.
Parts:
- removed C23: 100nF, Capacitor_SMD:C_0603_1608Metric, symbol Device:C
- removed R5: 1M, Resistor_SMD:R_0603_1608Metric, symbol Device:R_US
- removed R8: 17.8k, Resistor_SMD:R_0603_1608Metric, symbol Device:R_US
- removed U5: 74AUP1G74, Package_TO_SOT_SMD:SOT-23-5, symbol 74xGxx:74AUP1G74
- added R9: 0 Ω, Resistor_SMD:R_0603_1608Metric, symbol Device:R_US
- added TP5: BattMain, TestPoint:TestPoint_Pad_D1.0mm, symbol Connector:TestPoint
- added TP7: BuckEn, TestPoint:TestPoint_Pad_D1.0mm, symbol Connector:TestPoint
- BT1: value 9v Battery -> 4x AAA Batteries
Connections:
- net GND: now also C11.1, C14.2, U3.10 (GND2), U3.11 (GND2), U3.6 (GND1), U3.7 (GND1)
- net VBuckOut: now also R9.1; no longer C17.1, L1.2, TP2.1, U3.1 (Bias), U3.20 (Vout)
- net +9V renamed VBattMain
- net VBattMain: now also TP5.1
- net buck_en renamed pwr_buck_en
- net pwr_buck_en: now also TP7.1
- new net: C17.1, L1.2, R9.2, TP2.1, U3.1 (Bias), U3.20 (Vout)
- no-connect marks 2 -> 1
Other:
- moved on the sheet: C21
